Commit message: add dcamera & fixes. more custom scripts.

File: kortex_description/arms/gen3/6dof/urdf/gen3_macro.xacro (robot description, xacro)
@@ -257,52 +257,123 @@
         <child  link="${prefix}camera_color_frame" />
       </joint>
-      <!-- Simulated Camera Definition by Rishik -->
-      <link name="rishik_camera_link">
-        <visual>
-          <geometry>
-              <box size="0.01 0.005 0.005"/>
-          </geometry>
-          <material name="red"/>
-        </visual>
-      </link>
-      <joint name="rishik_camera_joint" type="fixed">
-        <parent link="${prefix}end_effector_link"/>
-        <child link="rishik_camera_link"/>
-        <origin xyz="0 0.05639 -0.00305" rpy="${-pi/2} ${-pi/2} 0" />
-      </joint>
-      <link name="rishik_camera_link_optical"></link>
-      <joint name="camera_optical_joint" type="fixed">
-        <parent link="rishik_camera_link"/>
-        <child link="rishik_camera_link_optical"/>
-        <origin xyz="0 0 0" rpy="${-pi/2} 0 ${-pi/2}"/>
-      </joint>
-      <gazebo reference="rishik_camera_link">
-        <material>Gazebo/Red</material>
-        <sensor name="camera" type="camera">
-          <pose> 0 0 0 0 0 0 </pose>
-          <visualize>true</visualize>
-          <update_rate>30</update_rate>
-          <camera>
-            <horizontal_fov>1.15</horizontal_fov>
-            <image>
-              <format>R8G8B8</format>
-              <width>640</width>
-              <height>480</height>
-            </image>
-            <clip>
-              <near>0.05</near>
-              <far>8.0</far>
-            </clip>
-            <noise>
-              <type>gaussian</type>
-              <mean>0.0</mean>
-              <stddev>0.007</stddev>
-            </noise>
-          </camera>
-          <plugin name="camera_controller" filename="libgazebo_ros_camera.so">
-              <frame_name>rishik_camera_link_optical</frame_name>
-          </plugin>
-        </sensor>
-      </gazebo>
+      <!-- Simulated Vision Definition by Rishik -->
+      <xacro:if value="${sim}">
+        <!-- COLOUR CAMERA -->
+        <link name="rishik_camera_link">
+          <visual>
+            <geometry>
+                <box size="0.01 0.005 0.005"/>
+            </geometry>
+            <material name="red"/>
+          </visual>
+        </link>
+        <joint name="rishik_camera_joint" type="fixed">
+          <parent link="${prefix}end_effector_link"/>
+          <child link="rishik_camera_link"/>
+          <origin xyz="0 0.05639 -0.00305" rpy="${-pi/2} ${-pi/2} 0" />
+        </joint>
+        <link name="rishik_camera_link_optical"></link>
+        <joint name="camera_optical_joint" type="fixed">
+          <parent link="rishik_camera_link"/>
+          <child link="rishik_camera_link_optical"/>
+          <origin xyz="0 0 0" rpy="${-pi/2} 0 ${-pi/2}"/>
+        </joint>
+        <gazebo reference="rishik_camera_link">
+          <material>Gazebo/Red</material>
+          <sensor name="camera" type="camera">
+            <pose> 0 0 0 0 0 0 </pose>
+            <visualize>true</visualize>
+            <update_rate>30</update_rate>
+            <camera>
+              <horizontal_fov>1.0821</horizontal_fov> <!-- FROM KINOVA MANUAL, pg 24 -->
+              <image>
+                <format>R8G8B8</format>
+                <width>1280</width>
+                <height>720</height>
+              </image>
+              <clip>
+                <near>0.03</near>
+                <far>8.0</far>
+              </clip>
+              <noise>
+                <type>gaussian</type>
+                <mean>0.0</mean>
+                <stddev>0.007</stddev>
+              </noise>
+            </camera>
+            <plugin name="camera_controller" filename="libgazebo_ros_camera.so">
+                <frameName>rishik_camera_link_optical</frameName>
+                <cameraName>camera/color</cameraName>
+                <imageTopicName>image_raw</imageTopicName>
+                <cameraInfoTopicName>camera_info</cameraInfoTopicName>
+            </plugin>
+          </sensor>
+        </gazebo>
+        <!-- DEPTH CAMERA -->
+        <link name="rishik_dcamera_link">
+          <visual>
+            <geometry>
+                <box size="0.01 0.005 0.005"/>
+            </geometry>
+            <material name="blue"/>
+          </visual>
+        </link>
+        <joint name="rishik_dcamera_joint" type="fixed">
+          <parent link="${prefix}end_effector_link"/>
+          <child link="rishik_dcamera_link"/>
+          <origin xyz="0 0.05639 -0.00305" rpy="${-pi/2} ${-pi/2} 0" />
+        </joint>
+        <link name="rishik_dcamera_link_optical"></link>
+        <joint name="dcamera_optical_joint" type="fixed">
+          <parent link="rishik_dcamera_link"/>
+          <child link="rishik_dcamera_link_optical"/>
+          <origin xyz="0 0 0" rpy="${-pi/2} 0 ${-pi/2}"/>
+        </joint>
+        <gazebo reference="rishik_dcamera_link">
+          <material>Gazebo/Blue</material>
+          <sensor name="openni_camera_camera" type="depth">
+            <always_on>1</always_on>
+            <visualize>true</visualize>
+            <update_rate>30</update_rate>
+            <pose> 0 0 0 0 0 0 </pose>
+            <camera>
+              <horizontal_fov>1.29154</horizontal_fov> <!-- FROM KINOVA MANUAL, pg 25 -->
+              <image>
+                <format>R8G8B8</format>
+                <width>480</width>
+                <height>270</height>
+              </image>
+              <clip>
+                <near>0.18</near> <!-- FROM KINOVA MANUAL, pg 25 -->
+                <far>1.5</far> <!-- EXPERIMENTAL ESTIMATE -->
+              </clip>
+              <noise>
+                <type>gaussian</type>
+                <mean>0.0</mean>
+                <stddev>0.007</stddev>
+              </noise>
+            </camera>
+            <plugin name="kinect" filename="libgazebo_ros_openni_kinect.so">
+              <frameName>rishik_dcamera_link/rishik_dcamera_link_optical</frameName>
+              <cameraName>camera/depth</cameraName>
+              <imageTopicName>image_raw</imageTopicName>
+              <depthImageTopicName>image</depthImageTopicName>
+              <depthImageCameraInfoTopicName>camera_info</depthImageCameraInfoTopicName>
+              <pointCloudTopicName>points</pointCloudTopicName>
+              <alwaysOn>true</alwaysOn>
+              <updateRate>30.0</updateRate>
+              <pointCloudCutoff>0.18</pointCloudCutoff>
+              <pointCloudCutoffMax>1.5</pointCloudCutoffMax>
+              <focalLength>0.0</focalLength>
+              <!-- <CxPrime>0</CxPrime> -->
+              <!-- <distortionK1>0.00000001</distortionK1>
+              <distortionK2>0.00000001</distortionK2>
+              <distortionK3>0.00000001</distortionK3>
+              <distortionT1>0.00000001</distortionT1>
+              <distortionT2>0.00000001</distortionT2> -->
+            </plugin>
+          </sensor>
+        </gazebo>
+      </xacro:if>
     </xacro:if>
   </xacro:macro>
